File: BrakeSwitch/BrakeSwitch.kicad_pcb (KiCad board)
At the start: 2 copper layers, 16 parts, among them Q1 NMOS, U1 XL1509-5.0, U2 LMV321, U3 LMV321

Commit message: Basic layout done
Parts:
- added C5: 1u, Capacitor_SMD:C_0603_1608Metric_Pad1.08x0.95mm_HandSolder, F.Cu at (114.2, 38.9)
- added C6: 1u, Capacitor_SMD:C_0603_1608Metric_Pad1.08x0.95mm_HandSolder, F.Cu at (114.2, 41.4)
- added J1: 12V_in, AA-Custom:SolderPad_01x02, B.Cu at (74.7, 48.8)
- added J2: LightPlug, AA-Custom:SolderPad_01x02, B.Cu at (74.7, 39.6)
- added J3: 5V_out, AA-Custom:SolderPad_01x02, B.Cu at (114.0, 56.9)
- added J4: Front_Pads, AA-Custom:SolderPad_01x03, B.Cu at (114.0, 48.5)
- added J5: Back_Pads, AA-Custom:SolderPad_01x03, B.Cu at (114.0, 38.6)
- added J6: 12V_in, AA-Custom:SolderPad_01x02, B.Cu at (74.7, 54.6)
- D2, D3, Q1, R4, R5, U2, U3: moved to B.Cu
- moved R5 53.4 mm to (78.0, 43.7), turned to -90 degrees
- moved R4 50.5 mm to (80.6, 42.9), turned to 180 degrees
- moved Q1 47.9 mm to (79.0, 39.6), turned to 90 degrees
- moved R1 32.2 mm to (95.0, 36.8)
- moved C2 26.0 mm to (78.3, 57.4), turned to 180 degrees
- moved D1 25.2 mm to (95.2, 42.9)
- moved U2 25.0 mm to (101.7, 45.6), turned to 90 degrees
- moved D2 24.6 mm to (97.3, 44.2), turned to -90 degrees
- moved U1 24.5 mm to (89.0, 41.2), turned to 90 degrees
- moved D3 24.4 mm to (104.4, 40.1)
- moved C4 22.8 mm to (78.4, 50.7), turned to 180 degrees
- moved C3 21.3 mm to (104.4, 41.7)
- moved U3 21.1 mm to (107.5, 45.6), turned to 90 degrees
- moved C1 15.4 mm to (78.4, 41.6), turned to 180 degrees
- moved RV1 15.1 mm to (102.4, 50.1)
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Other:
- board outline added: 43.9 x 26.4 mm

Commit message: Some feedback and layout
Parts:
- added H1: MountingHole, MountingHole:MountingHole_6.5mm_Pad, F.Cu at (92.7, 50.8)
- added RV2: Thresh, Potentiometer_THT:Potentiometer_Runtron_RM-065_Vertical, F.Cu at (78.8, 57.2)
- C5, C6, D1: moved to B.Cu
- J4: value Front_Pads -> Front_Loop
- J5: value Back_Pads -> Rear_Loop
- J6: value 12V_in -> 12V_Out
- moved J3 57.7 mm to (56.9, 49.3)
- moved J5 53.7 mm to (65.8, 62.2), turned to 180 degrees
- moved C5 42.7 mm to (71.6, 41.9), turned to -90 degrees
- moved J4 41.7 mm to (74.6, 62.2), turned to 180 degrees
- moved C6 41.1 mm to (73.2, 41.9), turned to -90 degrees
- moved U3 39.7 mm to (69.1, 55.4)
- moved D3 37.8 mm to (67.8, 49.6), turned to -90 degrees
- moved U2 29.2 mm to (74.2, 55.5)
- moved C3 28.2 mm to (76.2, 42.7)
- moved D1 27.4 mm to (67.8, 42.2), turned to 90 degrees
- moved R1 26.9 mm to (70.9, 48.8)
- moved D2 24.7 mm to (73.2, 49.6)
- moved RV1 23.7 mm to (78.8, 48.8)
- moved U1 22.6 mm to (66.9, 45.8)
- moved L1 21.4 mm to (70.9, 56.4), turned to -90 degrees
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Connections:
- C1 pad 1: /DCDC/Vin -> 12V
- C2 pad 1: /DCDC/Vin -> 12V
- C4 pad 1: /DCDC/Vin -> 12V
- U1 pad 1: /DCDC/Vin -> 12V
- U3 pad 3: Net-(U2--) -> Net-(U3--)
Other:
- board size 43.9 x 26.4 mm -> 47.8 x 26.4 mm
- board text added: "Diddy's Minion RIT Baja 3/19/2026"

Commit message: Progress save
Parts:
- added J2: Signal_Breakout, AA-Custom:SolderPad_01x04, F.Cu at (62.4, 67.9)
- added J7: Front_Brake_Switch, AA-Custom:SolderPad_01x02, F.Cu at (59.4, 71.9)
- added J8: Rear_Brake_Switch, AA-Custom:SolderPad_01x02, F.Cu at (59.4, 75.9)
- added J9: Light_In, AA-Custom:SolderPad_01x01, F.Cu at (69.3, 71.9)
- added SW1: AT SW-R2-2B-F-1-0, AA-Custom:SPDT_PanelMount_Switch, F.Cu at (82.9, 69.3)
Connections:
- C1 pad 2: GND -> SwitchF-
- C2 pad 2: GND -> SwitchF-
- C3 pad 2: GND -> SwitchF-
- C4 pad 2: GND -> SwitchF-
- C5 pad 2: GND -> SwitchF-
- C6 pad 2: GND -> SwitchF-
- D1 pad 2: GND -> SwitchF-
- J1 pad 2: GND -> SwitchF-
- J3 pad 1: GND -> SwitchF-
- J4 pad 3: GND -> SwitchF-
- J5 pad 3: GND -> SwitchF-
- J6 pad 2: GND -> SwitchF-
- Q1 pad 1: Light Out -> SwitchF-
- Q1 pad 2: Light Out -> SwitchF-
- Q1 pad 3: Light Out -> SwitchF-
- Q1 pad 5: Light In -> Net-(Q1-D)
- R1 pad 2: GND -> SwitchF-
- R5 pad 2: GND -> SwitchF-
- RV1 pad 3: GND -> SwitchF-
- RV2 pad 3: GND -> SwitchF-
- U1 pad 5: GND -> SwitchF-
- U1 pad 6: GND -> SwitchF-
- U1 pad 7: GND -> SwitchF-
- U1 pad 8: GND -> SwitchF-
- U2 pad 2: GND -> SwitchF-
- U3 pad 2: GND -> SwitchF-

Commit message: Laptop save
Parts:
- moved J2 9.78 mm to (52.6, 67.1)
Changed lines of the file:
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@@
 			(unlocked yes)
 			(layer "F.SilkS")
+			(hide yes)
 			(effects
 				(font
@@
 			(unlocked yes)
 			(layer "F.SilkS")
+			(hide yes)
 			(effects
 				(font
@@
 	(footprint "AA-Custom:SolderPad_01x04"
 		(layer "F.Cu")
-		(at 62.392 67.882)
+		(at 52.65 67.056)
 		(property "Reference" "J2"
 			(at 0 2.5 0)
 			(unlocked yes)
 			(layer "F.SilkS")
+			(hide yes)
 			(effects
 				(font
@@
 			(unlocked yes)
 			(layer "F.SilkS")
+			(hide yes)
 			(effects
 				(font
@@
 			(unlocked yes)
 			(layer "F.SilkS")
-			(effects
-				(font
+			(hide yes)
+			(effects
+				(font

Commit message: deskptop progress save
Parts:
- moved SW1 38.2 mm to (48.3, 53.4), turned to -90 degrees
- moved J2 21.0 mm to (35.7, 40.8)
- moved J1 21.0 mm to (35.9, 55.0)
- moved J3 21.0 mm to (35.9, 49.1)
- moved J6 21.0 mm to (35.9, 60.8)
- moved J4 15.9 mm to (87.5, 71.6)
- moved J5 15.9 mm to (78.7, 71.6)
Other:
- board size 47.8 x 26.4 mm -> 82.3 x 59.8 mm
Changed lines of the file:
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@@
 	(footprint "AA-Custom:SPDT_PanelMount_Switch"
 		(layer "F.Cu")
-		(at 82.916 69.342)
+		(at 48.26 53.355 -90)
 		(property "Reference" "SW1"
-			(at 0 4.5 0)
+			(at 0 4.5 270)
 			(unlocked yes)
 			(layer "F.SilkS")
@@
 		)
 		(property "Value" "AT SW-R2-2B-F-1-0"
-			(at 0 6 0)
+			(at 0 6 270)
 			(unlocked yes)
 			(layer "F.Fab")
@@
 		)
 		(property "Datasheet" "https://www.digikey.at/en/products/detail/adam-tech/SW-R2-2B-F-1-0/15284399"
-			(at 0 0 0)
+			(at 0 0 270)
 			(unlocked yes)
 			(layer "F.Fab")
@@
 		)
 		(property "Description" "Switch, single pole double throw"
-			(at 0 0 0)
+			(at 0 0 270)
 			(unlocked yes)
 			(layer "F.Fab")
@@
 		(sheetfile "BrakeSwitch.kicad_sch")
 		(attr smd)
+		(fp_rect
+			(start -9.4 -6.5)
+			(end 9.4 6.5)
+			(stroke
+				(width 0.1)
+				(type solid)
+			)
+			(fill no)
+			(layer "F.SilkS")
+		)
+		(fp_rect
+			(start -9.65 -6.75)
+			(end 9.65 6.75)
+			(stroke
+				(width 0.1)
+				(type solid)
+			)
+			(fill no)
+			(layer "F.CrtYd")
+		)
 		(fp_text user "${REFERENCE}"
-			(at 0 7.5 0)
+			(at 0 7.5 270)
 			(unlocked yes)
 			(layer "F.Fab")
@@
 		)
 		(pad "1" thru_hole oval
-			(at -7 0 180)
+			(at -7 0 90)
 			(size 3 7)
 			(drill oval 1 5)
@@
 		)
 		(pad "2" thru_hole oval
-			(at 0 0 180)
+			(at 0 0 90)
 			(size 3 7)
 			(drill oval 1 5)
@@
 		)
 		(pad "3" thru_hole oval
-			(at 7 0 180)
+			(at 7 0 90)
 			(size 3 7)
 			(drill oval 1 5)
@@
 		)
 		(embedded_fonts no)
+		(model "D:/Git/KiCadCustom/CadModels/RockerSwitchSPDT.step"
+			(offset
+				(xyz 0 0 14.5)
+			)
+			(scale
+				(xyz 1 1 1)
+			)
+			(rotate
+				(xyz -0 -0 -0)
+			)
+		)
 	)
 	(footprint "Potentiometer_THT:Potentiometer_Runtron_RM-065_Vertical"
@@
 	(footprint "AA-Custom:SolderPad_01x02"
 		(layer "B.Cu")
-		(at 56.896 55.118 90)
+		(at 35.941 54.991 90)
 		(property "Reference" "J1"
 			(at 0 2.54 90)
@@
 	(footprint "AA-Custom:SolderPad_01x02"
 		(layer "B.Cu")
-		(at 56.896 60.96 -90)
+		(at 35.941 60.833 -90)
 		(property "Reference" "J6"
 			(at 0 -2.5 90)
@@
 	(footprint "AA-Custom:SolderPad_01x03"
 		(layer "B.Cu")
-		(at 74.628 62.23 180)
+		(at 87.455 71.628 180)
 		(property "Reference" "J4"
 			(at 0 -2.5 0)
@@
 	(footprint "AA-Custom:SolderPad_01x03"
 		(layer "B.Cu")
-		(at 65.834 62.23 180)
+		(at 78.661 71.628 180)
 		(property "Reference" "J5"
 			(at 0 -2.5 0)
@@
 	(footprint "AA-Custom:SolderPad_01x02"
 		(layer "B.Cu")
-		(at 56.642 40.894 90)
+		(at 35.687 40.767 90)
 		(property "Reference" "J2"
 			(at 0 2.286 270)
@@
 	(footprint "AA-Custom:SolderPad_01x02"
 		(layer "B.Cu")
-		(at 56.896 49.276 90)
+		(at 35.941 49.149 90)
 		(property "Reference" "J3"
 			(at 3.556 0 270)
@@
 		(embedded_fonts no)
 	)
-	(gr_line
-		(start 92.71 42.672)
-		(end 93.472 39.116)
+	(gr_rect
+		(start 24.257 19.558)
+		(end 106.553 79.375)
 		(stroke
-			(width 2.54)
-			(type solid)
-		)
-		(layer "F.SilkS")
-	)
-	(gr_circle
-		(center 92.71 50.8)
-		(end 100.076 50.8)
-		(stroke
-			(width 1.016)
+			(width 0.2)
 			(type solid)
 		)
 		(fill no)
-		(layer "F.SilkS")
-	)
-	(gr_line
-		(start 92.837 58.928)
-		(end 93.599 62.484)
-		(stroke
-			(width 2.54)
-			(type solid)
-		)
-		(layer "F.SilkS")
-	)
-	(gr_line
-		(start 54.61 64.008)
-		(end 54.61 37.592)
-		(stroke
-			(width 0.1)
-			(type solid)
-		)
-		(layer "Edge.Cuts")
-	)
-	(gr_line
-		(start 82.804 37.592)
-		(end 54.61 37.592)
-		(stroke
-			(width 0.1)
-			(type solid)
-		)
-		(layer "Edge.Cuts")
-	)
-	(gr_curve
-		(pts
-			(xy 82.804 37.592) (xy 82.804 37.592) (xy 102.362 37.592) (xy 102.362 50.8)
-		)
-		(stroke
-			(width 0.127)
-			(type solid)
-		)
-		(layer "Edge.Cuts")
-	)
-	(gr_line
-		(start 82.804 64.008)
-		(end 54.61 64.008)
-		(stroke
-			(width 0.1)
-			(type solid)
-		)
-		(layer "Edge.Cuts")
-	)
-	(gr_curve
-		(pts
-			(xy 102.362 50.8) (xy 102.362 64.008) (xy 82.804 64.008) (xy 82.804 64.008)
-		)
-		(stroke
-			(width 0.127)
-			(type solid)
-		)
 		(layer "Edge.Cuts")
 	)

Commit message: Layout doneish
Parts:
- removed the J2 at (35.7, 40.8)
- C2, J7, J8, J9, R1, U1: moved to B.Cu
- moved J4 40.6 mm to (61.4, 40.5)
- moved J8 37.5 mm to (46.9, 40.5), turned to 180 degrees
- moved J9 35.6 mm to (42.2, 48.9), turned to 90 degrees
- moved J5 32.1 mm to (70.9, 40.5)
- moved J7 31.9 mm to (53.4, 40.5), turned to 180 degrees
- moved J2 26.8 mm to (48.1, 40.6)
- moved Q1 17.2 mm to (56.9, 60.2), turned to 180 degrees
- moved C6 13.9 mm to (67.8, 54.7)
- moved R5 13.1 mm to (64.5, 60.3), turned to 0 degrees
- moved C5 13.0 mm to (69.3, 54.7)
- moved R4 11.9 mm to (64.5, 58.8)
- moved R1 10.6 mm to (64.5, 57.3), turned to 180 degrees
- moved U3 10.5 mm to (75.2, 46.9), turned to -90 degrees
- moved D3 9.84 mm to (75.7, 55.5), turned to 90 degrees
- moved U2 9.08 mm to (71.7, 46.8), turned to -90 degrees
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Connections:
- net SwitchF- renamed GND
Other:
- board size 82.3 x 59.8 mm -> 60.2 x 25.8 mm

Commit message: Starting traces
Connections:
- J6 pad 1: 12V_out -> 12V
Routing:
- net 5V: track 0.00 -> 96.2 mm, vias 0 -> 4
- net 12V: track 0.00 -> 37.1 mm, vias 0 -> 3
- net RearLoop: track 0.00 -> 31.4 mm, vias 0 -> 1
- net FrontLoop: track 0.00 -> 23.7 mm, vias 0 -> 1
- net Net-(U3--): track 0.00 -> 16.7 mm
- net Net-(D1-K): track 0.00 -> 16.3 mm, vias 0 -> 2
- net SwitchF+: track 0.00 -> 13.7 mm
- net Net-(D2-K): track 0.00 -> 10.9 mm
- net Net-(U2--): track 0.00 -> 10.0 mm
- net Light In: track 0.00 -> 9.13 mm
- net Net-(Q1-G): track 0.00 -> 7.50 mm
- net Net-(D2-A): track 0.00 -> 5.71 mm
- net Net-(D3-A): track 0.00 -> 5.66 mm
- net Net-(U1-~{EN}): track 0.00 -> 2.21 mm

Commit message: Finished tracing
Parts:
- moved C5 1.80 mm to (67.6, 54.5), turned to 90 degrees
- moved R4 1.59 mm to (66.1, 58.8)
- moved C6 1.30 mm to (69.1, 54.5), turned to 90 degrees
- moved J5 0.81 mm to (70.1, 40.5)
- moved J4 0.46 mm to (61.0, 40.5)
- moved J8 0.30 mm to (47.2, 40.5)
- moved J7 0.10 mm to (53.3, 40.5)
- moved R1 0.06 mm to (64.5, 57.3)
- moved R5 0.06 mm to (64.5, 60.3), turned to 180 degrees
Routing:
- net GND: track 0.00 -> 74.2 mm, vias 0 -> 33
- net Net-(Q1-G): track 7.50 -> 11.3 mm
- net 5V: track 96.2 -> 99.5 mm, vias 4 -> 5
- net 12V: track 37.1 -> 34.3 mm
- net Net-(D2-K): track 10.9 -> 9.31 mm
- net RearLoop: track 31.4 -> 32.6 mm
- added copper zone on B.Cu, net 12V
- added copper zone on B.Cu, net GND
- added copper zone on F.Cu, net GND
- added copper zone on B.Cu, net Net-(Q1-D)
