File: BrakeSwitch/BrakeSwitch.kicad_pcb (KiCad board)
At the start: 2 copper layers, 60.2 x 25.8 mm, 30 parts, among them J1 12V_in, J2 Signal_Breakout, J3 5V_out, J4 Front_Loop, J5 Rear_Loop, J6 12V_Out, J7 Front_Brake_Switch, J8 Rear_Brake_Switch, J9 Light_In, Q1 NMOS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

Commit message: Done?
Other:
- board size 60.2 x 25.8 mm -> 62.5 x 25.9 mm
- board text added: "12Vin"
- board text added: "12Vout"
- board text added: "5V"
- board text added: "F"
- board text added: "GND"
- board text added: "LightIn"
- board text added: "R"
- board text added: "SwF"
- board text added: "SwR"
